File: _saved_Elemental-pHAT.sch (KiCad schematic (older format))
At the start: 53 parts, among them J1 GPIO4, J10 USB, J11 GPIO12, J12 S3, J13 A3, J14 JP_3.3V, J15 GPIO13, J16 S4, J17 A4, J18 CH5, J19 CH6, J2 S0, J20 CH7, J21 JP_5V, J22 I2C-1, J23 I2C-2, J24 SER6, J25 SER7, J26 SER8, J27 SER9, J28 SER10, J29 SER11, J3 A0, J4 GPIO5, J5 S1, J6 A1, J7 GPIO6, J8 S2, J9 A2, U1 Rpi3_Header, U2 AMS1117, U3 PCA9685, U4 MCP3008

Commit message: Esquema terminado
Parts:
- removed C1, C4: 22uF, symbol CP_Small
- removed C2, C3: 100nF, symbol C_Small
- removed D1: LED_PURPLE, symbol LED_Small
- removed J10: USB, symbol USB_A
- removed J14: JP_3.3V, symbol Conn_01x03_Male
- removed J21: JP_5V, symbol Conn_01x03_Male
- removed R1: 1k, symbol R_Small
- removed U2: AMS1117, SOT223, symbol V_REG_LM1117SOT223
- added J?: Jack-DC, symbol Jack-DC
- J?: renamed from J18; value CH5 -> Conn_01x01
- J?: renamed from J19; value CH6 -> Conn_01x01
- J?: renamed from J20; value CH7 -> Conn_01x01
- J?: renamed from J24; value SER6 -> Conn_01x01
- J?: renamed from J25; value SER7 -> Conn_01x01
- J?: renamed from J26; value SER8 -> Conn_01x01
- J?: renamed from J27; value SER9 -> Conn_01x01
- J?: renamed from J28; value SER10 -> Conn_01x01
- J?: renamed from J29; value SER11 -> Conn_01x01
- renumbered C5 to C?, J3 to J?, J22 to J?, J6 to J?, J9 to J?, J13 to J?, J2 to J?, J5 to J?, J8 to J?, J12 to J?, J17 to J?, J16 to J?, J23 to J?, J1 to J?, J4 to J?, J7 to J?, J11 to J?, J15 to J?, JP1 to JP?, JP2 to JP?, JP3 to JP?, JP4 to JP?, JP5 to JP?, JP6 to JP?, R2 to R?, R3 to R?, R4 to R?, R5 to R?, R6 to R?, R7 to R?, R8 to R?, U1 to U?, U3 to U?, U4 to U?
Connections:
- net 3V3RPI is gone; now on net +3V3: U?.1 (3.3V), U?.17 (3.3V)
- net 5VRPI: no longer names the net of U?.2 (5V)
- net 5VRPI: no longer U?.4 (5V)
- no-connect marks 8 -> 0
