File: Elemental-pHAT.kicad_pcb (KiCad board)
At the start: 2 copper layers, 65 x 30 mm, 47 parts, among them J1 GPIO4, J10 USB, J11 GPIO12, J12 S3, J13 A3, J14 JP_3.3V, J15 GPIO13, J16 S4, J17 A4, J18 CH5, J19 CH6, J2 S0, J21 JP_5V, J22 I2C-1, J24 SER6, J25 SER7, J3 A0, J4 GPIO5, J5 S1, J6 A1, J7 GPIO6, J8 S2, J9 A2, U1 Rpi3_Header, U2 AMS1117, U3 PCA9685, U4 MCP3008

Commit message: Routed
Parts:
- moved R1 45.3 mm to (154.6, 98.4)
- moved D1 45.2 mm to (154.6, 96.5)
- moved J21 19.2 mm to (114.8, 105.2)
- moved J14 18.5 mm to (114.8, 107.8)
- moved J18 5.72 mm to (127.4, 106.3)
- moved J10 3.43 mm to (109.9, 99.2)
- moved C3 2.67 mm to (116.3, 101.6)
- moved C2 2.41 mm to (116.3, 97.2)
- moved U4 2.01 mm to (125.0, 100.2)
- moved J1 1.52 mm to (151.9, 110.1)
- moved J11 1.52 mm to (160.3, 110.1)
- moved J15 1.52 mm to (163.1, 110.1)
- moved J4 1.52 mm to (154.7, 110.1)
- moved J7 1.52 mm to (157.5, 110.1)
- moved C5 0.76 mm to (137.4, 99.7)
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Routing:
- net GND: track 0.00 -> 136.9 mm, vias 0 -> 1
- net +3V3: track 0.00 -> 126.1 mm, vias 0 -> 3
- net +5V: track 0.00 -> 89.8 mm, vias 0 -> 2
- net /SCL: track 0.00 -> 78.2 mm, vias 0 -> 2
- net /SDA: track 0.00 -> 77.6 mm, vias 0 -> 2
- net /GPIO4: track 0.00 -> 43.9 mm
- net /3V3RPI: track 0.00 -> 41.5 mm
- net /GPIO6: track 0.00 -> 38.9 mm, vias 0 -> 1
- net /GPIO12: track 0.00 -> 37.4 mm
- net /A0: track 0.00 -> 32.1 mm, vias 0 -> 3
- net /A1: track 0.00 -> 29.6 mm, vias 0 -> 3
- net /A2: track 0.00 -> 28.0 mm, vias 0 -> 3
- net /A3: track 0.00 -> 27.5 mm, vias 0 -> 3
- net /A4: track 0.00 -> 26.8 mm, vias 0 -> 3
- net /3V3USB: track 0.00 -> 26.1 mm
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- added copper zone on B.Cu, net GND
- added copper zone on F.Cu, net GND

Commit message: Silkscreen finished
Parts:
- added G***: LOGO, logos_frizzy:web, B.Cu at (171.6, 103.5)
- moved J19 0.74 mm to (130.6, 105.7)
- moved J18 0.68 mm to (127.6, 105.7)
- renumbered JP1 to A0, JP2 to A1, JP3 to A2, JP4 to A3, JP5 to A4, JP6 to A5, J22 to I2C
Routing:
- net GND: track 136.9 -> 152.0 mm, vias 1 -> 4
- net (no net): track 0.00 -> 3.12 mm, vias 0 -> 9
- net /CH5: track 3.61 -> 3.08 mm
Other:
- board text added: "A0"
- board text added: "A1"
- board text added: "A2"
- board text added: "A3"
- board text added: "A4"
- board text added: "A5"
- board text added: "A6"
- board text added: "GPIO12"
- board text added: "GPIO13"
- board text added: "GPIO4"
- board text added: "GPIO5"
- board text added: "GPIO6"
- board text added: "I2C - 3V3"
- board text added: "ON"
- board text added: "PWD IN^"
- board text added: "S0"
- board text added: "S1"
- board text added: "S2"
- board text added: "S3"
- board text added: "S4"
- board text added: "SER6"
- board text added: "SER7"
- board text added: "USB|3.3V|RPI"
- board text added: "USB|5V|RPI"
